File: keypoint/untitled.sch (EAGLE design)
At the start: 66 parts, among them J3 10103594, K1 351, K2 351, Q1 MMBT3904, Q2 MMBT3904, Q3 12MHz, Q4 S9013, Q5 S9013, U1 AMS1117, U2 MAX232CSE, U3 PC817X2NIP0F, U4 PC817X2NIP0F, U5 MAX232CSE, X1 MSTBA2, X2 MSTBA3

Commit message: fix PCB versi 1.0
Parts:
- removed D8: US1M-13, US1M-13:US1M-13
- removed K2: 351, relay:351
- removed Q5: S9013, S9013:S9013
- removed R11: 330, adafruit:R-US_M0805
- removed R14: 1k, adafruit:R-US_M0805
- removed U4: PC817X2NIP0F, PC817X2NIP0F:PC817X2NIP0F
- added D10, D11, D9: US1M-13, US1M-13:US1M-13
- added R15, R16, R17: 10K, adafruit:R-US_M0805
- R4, R5: value 1K -> 10K
Connections:
- removed net N$30: R11.2, U4.A
- removed net N$31: R14.1, U4.CT
- removed net N$33: D8.A, K21.2, Q5.C
- removed net N$36: Q5.B, U4.ET
- removed net RXLORA_CONFIG: K23.S, X2-2.1
- removed net TXLORA_CONFIG: K22.S, X2-3.1
- new net N$38: D9.K, U5.R2OUT
- new net N$39: D10.K, U2.R2OUT
- new net N$40: D11.K, EBYTEE220-900T22D1.TXD
- new net SCL: MD1.IO22, X2-2.1
- new net SDA: MD1.IO21, X2-3.1
- net 3V3: now also R15.2, R16.2, R17.2
- net GND: no longer Q5.E, U4.C
- net OUT+: no longer D8.K, K21.1, R14.2
- net RXLORA: now also D5.A, K12.O, R6.1; no longer K23.P
- net RX_DB9: now also D9.A, K12.P, R15.1; no longer K13.P, K22.O, MD1.IO16, U5.R2OUT
- net RX_DB9-1: now also D10.A, R16.1; no longer U2.R2OUT
- net SW_LORACONFIG: no longer R11.1
- net TXLORA: now also D11.A, K13.O, MD1.IO16, R17.1; no longer EBYTEE220-900T22D1.TXD, K22.P
- net TX_DB9: now also K13.P; no longer D5.A, K12.P, K23.O, R6.1
