File: keypoint v1.0/untitled.brd (EAGLE design)
At the start: 88 x 60 mm, 66 parts, among them J3 10103594, K1 351, Q1 MMBT3904, Q2 MMBT3904, Q3 12MHz, Q4 S9013, U1 AMS1117, U2 MAX232CSE, U3 PC817X2NIP0F, U5 MAX232CSE, X1 MSTBA2, X2 MSTBA3

Commit message: fix PCB version 1.0
Parts:
- R4, R5: value 1K -> 10K
- moved R9 17.6 mm to (17.5, 50.2)
- moved U3 3.35 mm to (12.3, 45.3), turned to 270 degrees
- moved R1 0.76 mm to (7.89, 38.1)
- moved R2 0.76 mm to (7.91, 35.9)
Routing:
- net GND: track 351.4 -> 368.7 mm
- net SW_MODEM: track 112.0 -> 128.7 mm
- net N$29: track 105.6 -> 116.6 mm
- net N$18: track 3.07 -> 10.6 mm
- net RTS: track 70.5 -> 66.6 mm
- net N$16: track 10.1 -> 12.1 mm
- net N$6: track 30.8 -> 32.5 mm
- net OUT+: track 188.1 -> 189.2 mm
- net DTR: track 63.5 -> 64.1 mm
- removed copper zone on layer 16, net GROUNDING
Other:
- outline, holes or cut-outs redrawn
- board text added: "Version 1.0"
