File: keypoint v1.0/untitled.sch (EAGLE design)
At the start: 72 parts, among them J3 10103594, K1 351, K2 351, Q1 MMBT3904, Q2 MMBT3904, Q3 12MHz, Q4 S9013, Q5 S9013, U1 AMS1117, U2 MAX232CSE, U3 PC817X2NIP0F, U4 PC817X2NIP0F, U5 MAX232CSE, X1 MSTBA2, X2 MSTBA3

Commit message: fix PCB version 1.0
Parts:
- removed D8: US1M-13, US1M-13:US1M-13
- removed K2: 351, relay:351
- removed Q5: S9013, S9013:S9013
- removed R11: 330, adafruit:R-US_M0805
- removed R14: 1k, adafruit:R-US_M0805
- removed U4: PC817X2NIP0F, PC817X2NIP0F:PC817X2NIP0F
- R4, R5: value 1K -> 10K
Connections:
- removed net N$30: R11.2, U4.A
- removed net N$31: R14.1, U4.CT
- removed net N$33: D8.A, K21.2, Q5.C
- removed net N$36: Q5.B, U4.ET
- removed net N$37: K23.O
- removed net RXLORA_CONFIG: K23.S, X2-2.1
- removed net TXLORA_CONFIG: K22.S, X2-3.1
- new net SCL: MD1.IO22, X2-2.1
- new net SDA: MD1.IO21, X2-3.1
- net GND: no longer Q5.E, U4.C
- net OUT+: no longer D8.K, K21.1, R14.2
- net RXLORA: now also D5.A, R6.1; no longer K23.P
- net SW_LORACONFIG: no longer R11.1
- net TXLORA: no longer K22.O, K22.P
- net TX_DB9: no longer D5.A, R6.1
